File: BENOTL-HW/Robot/talentBadge.kicad_pcb (KiCad board)
At the start: 2 copper layers, 62 parts, among them P1 USB_A, P2 OLED, P3 Batt, P4 PS, P5 sd_card_spi, Q1 MMBT3904, Q2 MMBT3904, Q3 IR phototransistor, SW1 B1, SW2 B2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

Commit message: Changes Tesla  Layout Files
Parts:
- added svg2mod: G***, Robot:Robot_Edge.Cuts.mod, F.Cu at (75.3, 104.7)
Other:
- board outline added: 93.8 x 102.7 mm
