File: BENOTL-HW/Robot/talentBadge.kicad_pcb (KiCad board)
At the start: 2 copper layers, 93.8 x 102.7 mm, 65 parts, among them P1 USB_A, P2 OLED, P3 Batt, P4 PS, P5 sd_card_spi, Q1 MMBT3904, Q2 MMBT3904, Q3 IR phototransistor, SW1 B1, SW2 B2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

Commit message: Agregado logos robot
Parts:
- added G***: LOGO, talentBadgelogo:espressif_logo, B.Cu at (60.7, 105.9)
- added G***: LOGO, talentBadgelogo:pcbway_logo, B.Cu at (69.3, 120.9)

Commit message: medio fixes
Routing:
- net +3V3: track 387.3 -> 416.0 mm, vias 11 -> 12
- net GND: track 271.3 -> 283.8 mm, vias 17 -> 19
- net Net-(U5-Pad2): track 31.9 -> 42.0 mm
- net RST: track 120.2 -> 128.9 mm
- net np2: track 11.1 -> 14.4 mm
- net Net-(C3-Pad1): track 38.2 -> 36.0 mm
- net Net-(Q1-Pad1): track 6.28 -> 7.46 mm
- net DTR: track 18.1 -> 19.2 mm
- net Net-(U7-Pad2): track 32.0 -> 33.0 mm
- net GPIO0: track 52.3 -> 53.3 mm
- net RTS: track 9.13 -> 9.92 mm
- net Net-(Q2-Pad1): track 4.98 -> 5.63 mm

Commit message: Agregado logos Wurth y Makers a Robot
Parts:
- added G***: LOGO, talentBadgeLogo:makers_logo, B.Cu at (72.4, 144.0)
- added G***: LOGO, talentBadgeLogo:wurth_logo, B.Cu at (74.9, 125.7)
- moved G*** 5.11 mm to (68.8, 115.8)
