File: BENOTL-HW/Cat/talentBadge.kicad_pcb (KiCad board)
At the start: 2 copper layers, 93.8 x 102.7 mm, 64 parts, among them P1 USB_A, P2 OLED, P3 Batt, P4 PS, P5 sd_card_spi, Q1 MMBT3904, Q2 MMBT3904, Q3 IR phototransistor, SW1 B1, SW2 B2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

Commit message: Changes Robot Layout files
Parts:
- removed svg2mod: G***, Robot:Robot_Edge.Cuts.mod
- removed svg2mod: G***, Robot:Robot_SilkS.mod
Other:
- board outline removed

Commit message: Changes Cat Layout files
Parts:
- added svg2mod: G***, Cat:Cat_Edge.Cuts.mod, F.Cu at (68.5, 110.3)
- added svg2mod: G***, Cat:Cat_SilkS.mod, F.Cu at (69.3, 111.4)
Other:
- board outline added: 80.5 x 102.9 mm
